File: XT-IDE.kicad_pcb (KiCad board)
At the start: 2 copper layers, 104.8 x 91.9 mm, 51 parts, among them J1 Power output, J2 XT-Slot8 Jumper, J3 External LED, J4 5V on IDE Pin20, J5 IDE IRQ, P6 CONN_1, P7 CONN_1, SW1 DIPS_06, SW2 DIPS_04, SW3 DPDT, SW4 DPDT, SW5 SPDT, SW6 SPDT, U1 74HCT573, U10 74HCT688, U11 74HCT245, U12 74LS33, U2 74HCT573, U3 74HCT245, U4 74HCT04, U5 74HCT32, U6 74HCT04, U7 74HCT138, U8 74HCT688, U9 28C256

Commit message: Add files via upload
Update files to Rev5.1
Parts:
- C1, C10, C11, C2, C3, C4, C5, C6, C7, C8, C9: footprint Capacitors_THT:C_Axial_L3.8mm_D2.6mm_P7.50mm_Horizontal -> Capacitors_THT:C_Rect_L7.0mm_W2.0mm_P5.00mm
- C13: footprint Capacitors_SMD:C_0805_HandSoldering -> Resistors_SMD:R_0805_HandSoldering
- J2: value XT-Slot8 Jumper -> Conn_01x02
- J4: value 5V on IDE Pin20 -> Conn_01x02
- J5: value IDE IRQ -> Conn_02x05_Odd_Even
- SW3: footprint Custom:CKCOMP-OS203011MS1QP1 -> Custom:CKCOMP-OS202011MA0QS1
- moved R2 26.3 mm to (200.7, 75.9)
- moved J3 3.43 mm to (204.5, 77.2)
- moved D1 3.18 mm to (197.5, 70.2)
- moved C8 1.58 mm to (133.6, 109.6)
- moved J1 1.52 mm to (117.7, 143.5)
- moved J5 1.49 mm to (121.4, 145.9)
- moved C4 1.37 mm to (165.1, 81.2)
- moved C7 1.37 mm to (199.4, 78.6)
- moved C3 1.37 mm to (152.4, 73.5)
- moved C5 1.37 mm to (176.5, 81.2)
- moved C1 1.37 mm to (127.0, 73.5)
- moved C10 1.37 mm to (191.5, 109.7)
- moved C11 1.37 mm to (203.6, 109.7)
- moved C2 1.37 mm to (139.7, 73.5)
- moved C6 1.37 mm to (188.0, 81.2)
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Connections:
- IDE1 pad 21: Net-(IDE1-Pad21) -> (no net)
- IDE1 pad 27: Net-(IDE1-Pad27) -> (no net)
- IDE1 pad 32: Net-(IDE1-Pad32) -> (no net)
- IDE1 pad 34: Net-(IDE1-Pad34) -> (no net)
- RP1 pad 2: Net-(RP1-Pad2) -> (no net)
- SW4 pad 3: Net-(SW4-Pad3) -> (no net)
- SW4 pad 6: Net-(SW4-Pad6) -> (no net)
- SW5 pad 3: Net-(SW5-Pad3) -> (no net)
- SW6 pad 3: Net-(SW6-Pad3) -> (no net)
- U12 pad 13: Net-(U12-Pad13) -> (no net)
- U7 pad 11: Net-(U7-Pad11) -> (no net)
- U7 pad 12: Net-(U7-Pad12) -> (no net)
- U7 pad 15: Net-(U7-Pad15) -> (no net)
- U7 pad 7: Net-(U7-Pad7) -> (no net)
Routing:
- net GND: track 324.6 -> 260.8 mm, vias 2 -> 1
- net IDE-A0: track 95.7 -> 60.0 mm, vias 1 -> 0
- net IOW: track 116.7 -> 141.3 mm
- net D9: track 91.6 -> 69.5 mm, vias 1 -> 0
- net VCC: track 430.3 -> 409.2 mm, vias 0 -> 1
- net CS_IDE: track 123.6 -> 143.1 mm, vias 2 -> 3
- net IDE-A2: track 53.0 -> 71.7 mm, vias 2 -> 0
- net Net-(J3-Pad2): track 24.2 -> 6.88 mm
- net A18: track 79.8 -> 63.4 mm, vias 2 -> 0
- net CS3FX: track 35.7 -> 52.1 mm, vias 0 -> 1
- net DB0: track 94.2 -> 110.2 mm, vias 1 -> 4
- net A6: track 74.2 -> 60.1 mm
- net A17: track 60.5 -> 74.5 mm
- net DB1: track 94.6 -> 108.3 mm, vias 0 -> 4
- net Net-(SW3-Pad5): track 74.9 -> 61.6 mm, vias 1 -> 0
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- added copper zone on F.Cu, net VCC
Other:
- board size 104.8 x 91.9 mm -> 105.7 x 96 mm
- net class Default: clearance 0.2032 -> 0.2; trace_width 0.2032 -> 0.2
- net class Power: clearance 0.2032 -> 0.2; trace_width 1 -> 0.8; via_dia 1 -> 0.8; via_drill 0.5 -> 0.4
- rule trace_clearance: 0.2032 -> 0.2
- rule trace_min: 0.2 -> 0.127
- board text added: "HiSpeed Mode"
- board text added: "IDE IRQ isn't supported in XT-IDE Universal BIOS as of R598. Leave unjumpered."
- board text added: "Monotech XT-IDE 8-bit ISA IDE Interface + Boot ROM"
- board text added: "ROM Enable"
- board text added: "ROM Write-Enable"
- board text added: "Rev 5.1"
- board text removed: "< CMPT"
- board text removed: "<EN"
- board text removed: "<WE"
- board text removed: "Compatibility Mode"
- board text removed: "HiSpeed <-> Compat"
- board text removed: "I D E"
- board text removed: "IDE IRQ isn't supported in XT-IDE Universal BIOS as of May 2018. Leave unjumpered."
- board text removed: "Monotech XT-IDE - 8-bit ISA IDE Interface + Boot ROM"
- board text removed: "R O M"
- board text removed: "Rev 5"

Commit message: Add files via upload
Parts:
- C1, C10, C11, C13, C2, C3, C4, C5, C6, C7, C8, C9: value C -> 0.1uF
- IDE1: footprint Custom:Pin_Header_Angled_2x20_ShortSilkS -> Custom:Pin_Header_Angled_2x20_Pitch2.54mm_Shrouded
- RP1, RP2: value 10k -> 10K
- SW1: value DIPS_06 -> IDE Address; footprint Buttons_Switches_THT:SW_DIP_x6_W7.62mm_Slide -> Buttons_Switches_THT:SW_DIP_x6_W7.62mm_Slide_LowProfile
- SW2: value DIPS_04 -> ROM Address; footprint Buttons_Switches_THT:SW_DIP_x4_W7.62mm_Slide -> Buttons_Switches_THT:SW_DIP_x4_W7.62mm_Slide_LowProfile
- U9: value 28C256 -> 28C64B/28C256
- moved REF*** 82.5 mm to (204.6, 117.0)
- moved U7 68.2 mm to (147.3, 131.8), turned to 270 degrees
- moved J2 63.5 mm to (202.6, 129.3)
- moved G*** 61.1 mm to (134.0, 146.9)
- moved C8 60.7 mm to (190.1, 87.4), turned to 90 degrees
- moved SW1 60.2 mm to (154.9, 68.7), turned to 270 degrees
- moved SW2 52.6 mm to (177.4, 68.7), turned to 270 degrees
- moved SW6 50.7 mm to (134.8, 72.3)
- moved C10 50.4 mm to (149.9, 138.2), turned to 90 degrees
- moved U11 50.3 mm to (147.3, 106.4)
- moved SW5 48.0 mm to (126.0, 72.3)
- moved RP1 45.8 mm to (157.5, 78.5), turned to 180 degrees
- moved R3 42.1 mm to (181.2, 73.9)
- moved R4 41.9 mm to (181.2, 71.0)
- moved SW4 41.7 mm to (201.7, 103.8), turned to 180 degrees
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Connections:
- RP1 pad 2: (no net) -> Net-(RP1-Pad2)
- RP1 pad 8: Net-(RP1-Pad8) -> (no net)
- SW1 pad 10: Net-(RP1-Pad5) -> Net-(RP1-Pad4)
- SW1 pad 11: Net-(RP1-Pad4) -> Net-(RP1-Pad3)
- SW1 pad 12: Net-(RP1-Pad3) -> Net-(RP1-Pad2)
- SW1 pad 7: Net-(RP1-Pad8) -> Net-(RP1-Pad7)
- SW1 pad 8: Net-(RP1-Pad7) -> Net-(RP1-Pad6)
- SW1 pad 9: Net-(RP1-Pad6) -> Net-(RP1-Pad5)
- SW6 pad 1: ROM_WE -> (no net)
- SW6 pad 3: (no net) -> ROM_WE
- U8 pad 14: Net-(RP1-Pad8) -> Net-(RP1-Pad7)
- U8 pad 16: Net-(RP1-Pad7) -> Net-(RP1-Pad6)
- U8 pad 18: Net-(RP1-Pad6) -> Net-(RP1-Pad5)
- U8 pad 3: Net-(RP1-Pad3) -> Net-(RP1-Pad2)
- U8 pad 5: Net-(RP1-Pad4) -> Net-(RP1-Pad3)
- U8 pad 7: Net-(RP1-Pad5) -> Net-(RP1-Pad4)
Routing:
- net A0: track 138.7 -> 239.7 mm
- net D4: track 140.8 -> 42.5 mm
- net D5: track 138.5 -> 42.5 mm
- net A4: track 55.0 -> 150.3 mm
- net D3: track 137.8 -> 42.5 mm
- net D6: track 134.9 -> 41.4 mm, vias 1 -> 0
- net D2: track 135.5 -> 42.5 mm
- net D0: track 134.5 -> 42.5 mm
- net D1: track 134.5 -> 42.5 mm
- net A5: track 56.2 -> 146.4 mm
- net A6: track 60.1 -> 150.3 mm, vias 1 -> 2
- net A8: track 76.8 -> 161.1 mm, vias 2 -> 0
- net A7: track 73.0 -> 156.3 mm, vias 2 -> 0
- net A9: track 86.8 -> 160.4 mm
- net IOW: track 141.3 -> 73.0 mm, vias 3 -> 1
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- added copper zone on F.Cu, net GND
- removed copper zone on F.Cu, net VCC
Other:
- outline, holes or cut-outs redrawn
- net class Power: trace_width 0.8 -> 0.5; via_dia 0.8 -> 0.6; via_drill 0.4 -> 0.3
- board text added: "1 000011111111 2 111100001111 3 001100110011 4 010101010101"
- board text added: "1 0011111111111111111111111111111111 2 1100000000000000001111111111111111 3 0100000000111111110000000011111111 4 1100001111000011110000111100001111 5 1100110011001100110011001100110011 6 1101010101010101010101010101010101"
- board text added: "1 2 3 4"
- board text added: "1 2 3 4 5 6"
- board text added: "1 4"
- board text added: "1 6"
- board text added: "28C256 32K"
- board text added: "28C64B 8K"
- board text added: "7 5 4 3 2"
- board text added: "<ROM Enable"
- board text added: "<ROM Write-Protect"
- board text added: "=32KiB ROM Support"
- board text added: "Boot ROM"
- board text added: "Enable the ROM Write-Protect once system is up and running the way intended, to prevent accidental re-flashing."
- board text added: "HiSpeed Mode>"
- board text added: "IDE Address"
- board text added: "IDE Address Switch Settings"
- board text added: "Monotech XT-IDE Bootable 8-bit ISA IDE Interface"
- board text added: "ROM Address"
- board text added: "ROM Address Switch Settings"
- board text added: "ROM Chip Type"
- board text added: "Rev 5.2"
- board text removed: "0.1uF"
- board text removed: "10K"
- board text removed: "16 000011111111 15 111100001111 14 001100110011 13 010101010101"
- board text removed: "16 15 14 13"
- board text removed: "1K"
- board text removed: "2 3 4 5 7"
- board text removed: "28-pin EEPROM Socket"
- board text removed: "28C256"
- board text removed: "28C64B"
- board text removed: "47 - 100uF"
- board text removed: "74HCT04"
- board text removed: "74HCT138"
- board text removed: "74HCT245"
- board text removed: "74HCT32"
- board text removed: "74HCT573"
- board text removed: "74HCT688"
- board text removed: "74LS33"
- board text removed: "9 0011111111111111111111111111111111 8 1100000000000000001111111111111111 7 0100000000111111110000000011111111 6 1100001111000011110000111100001111 5 1100110011001100110011001100110011 4 1101010101010101010101010101010101"
- board text removed: "9 8 7 6 5 4"
- board text removed: "=32KB ROM Support"
- board text removed: "BIOS I/O Port"
- board text removed: "Boot ROM Enable"
- board text removed: "Boot ROM I/O Address Switch Settings"
- board text removed: "Boot ROM Write Enable"
- board text removed: "DIP Switch x4"
- board text removed: "DIP Switch x6"
- board text removed: "DIS <-> EN"
- board text removed: "Disable the "write-enable" once system is up and running the way intended, to prevent accidental re-flashing."
- board text removed: "EEPROM Type"
- board text removed: "EN <-> DIS"
- board text removed: "HiSpeed Mode"
- board text removed: "IDE I/O Address Switch Settings"
- board text removed: "IDE I/O Port"
- board text removed: "IDE Pin 1"
- board text removed: "Monotech XT-IDE 8-bit ISA IDE Interface + Boot ROM"
- board text removed: "ROM Enable"
- board text removed: "ROM Write-Enable"
- board text removed: "Refer to back for I/O Port switch settings"
- board text removed: "Rev 5.1"
- board text removed: "^ +5V ^"
- board text removed: "^ ^"

Commit message: Add files via upload
Parts:
- SW1: footprint Buttons_Switches_THT:SW_DIP_x6_W7.62mm_Slide_LowProfile -> Buttons_Switches_THT:SW_DIP_x6_W7.62mm_Slide
- SW2: footprint Buttons_Switches_THT:SW_DIP_x4_W7.62mm_Slide_LowProfile -> Buttons_Switches_THT:SW_DIP_x4_W7.62mm_Slide

Commit message: Updated to Rev5.3
Parts:
- removed the G*** at (134.0, 146.9)
- removed REF***: OSHW-Logo_11.4x12mm_SilkScreen, Symbols:OSHW-Logo_11.4x12mm_SilkScreen
- added C14: 10uF, Capacitor_THT:CP_Radial_Tantal_D4.5mm_P5.00mm, F.Cu at (113.5, 131.2)
- added G***: LOGO, Custom KiCad Library:Monotech Logo 18mm, F.Cu at (178.7, 144.5)
- C1, C10, C11, C2, C3, C4, C5, C6, C7, C8, C9: value 0.1uF -> 100nF; footprint Capacitors_THT:C_Rect_L7.0mm_W2.0mm_P5.00mm -> Capacitor_THT:C_Disc_D4.3mm_W1.9mm_P5.00mm
- C12: value 47uF -> 100nF; footprint Capacitors_THT:CP_Radial_D6.3mm_P2.50mm -> Capacitor_SMD:C_0805_2012Metric_Pad1.15x1.40mm_HandSolder; moved to B.Cu
- C13: value 0.1uF -> 10uF; footprint Resistors_SMD:R_0805_HandSoldering -> Capacitor_THT:CP_Radial_Tantal_D4.5mm_P5.00mm; moved to F.Cu
- D1: footprint LEDs:LED_D5.0mm -> LED_THT:LED_D5.0mm
- J1: footprint Pin_Headers:Pin_Header_Angled_1x04_Pitch2.54mm -> Connector_PinHeader_2.54mm:PinHeader_1x04_P2.54mm_Horizontal
- J2: footprint Pin_Headers:Pin_Header_Straight_1x02_Pitch2.54mm -> Jumper:SolderJumper-2_P1.3mm_Bridged_RoundedPad1.0x1.5mm
- J3: footprint Pin_Headers:Pin_Header_Angled_1x02_Pitch2.54mm -> Connector_PinHeader_2.54mm:PinHeader_1x02_P2.54mm_Horizontal
- J4: footprint Pin_Headers:Pin_Header_Straight_1x02_Pitch2.54mm -> Connector_PinHeader_2.54mm:PinHeader_1x02_P2.54mm_Vertical
- J5: footprint Pin_Headers:Pin_Header_Straight_2x05_Pitch2.54mm -> Connector_PinHeader_2.54mm:PinHeader_2x05_P2.54mm_Vertical
- P6, P7: footprint Mounting_Holes:MountingHole_3mm -> MountingHole:MountingHole_3.2mm_M3
- R1, R2, R3, R4: footprint Resistors_THT:R_Axial_DIN0207_L6.3mm_D2.5mm_P7.62mm_Horizontal -> Resistor_THT:R_Axial_DIN0207_L6.3mm_D2.5mm_P7.62mm_Horizontal
- R5, R6: value 10k -> 10K; footprint Resistors_SMD:R_0805_HandSoldering -> Resistor_SMD:R_0805_2012Metric_Pad1.15x1.40mm_HandSolder
- RP1, RP2: footprint Resistors_THT:R_Array_SIP8 -> Resistor_THT:R_Array_SIP9
- SW1: footprint Buttons_Switches_THT:SW_DIP_x6_W7.62mm_Slide -> Button_Switch_THT:SW_DIP_SPSTx06_Slide_9.78x17.42mm_W7.62mm_P2.54mm
- SW2: footprint Buttons_Switches_THT:SW_DIP_x4_W7.62mm_Slide -> Button_Switch_THT:SW_DIP_SPSTx04_Slide_9.78x12.34mm_W7.62mm_P2.54mm
- SW5, SW6: footprint Custom:CKCOMP-OS102011MA1QN1 -> Button_Switch_THT:SW_CuK_OS102011MA1QN1_SPDT_Angled
- U1, U2: value 74HCT573 -> 74LS573; footprint Housings_DIP:DIP-20_W7.62mm -> Custom KiCad Library:DIP-20_W7.62mm
- U10, U8: value 74HCT688 -> 74LS688; footprint Housings_DIP:DIP-20_W7.62mm -> Custom KiCad Library:DIP-20_W7.62mm
- U11, U3: value 74HCT245 -> 74LS245; footprint Housings_DIP:DIP-20_W7.62mm -> Custom KiCad Library:DIP-20_W7.62mm
- U12: footprint Housings_SOIC:SOIC-14_3.9x8.7mm_Pitch1.27mm -> Custom KiCad Library:SOIC-14_3.9x8.7mm_P1.27mm
- U4, U6: value 74HCT04 -> 74LS04; footprint Housings_DIP:DIP-14_W7.62mm -> Custom KiCad Library:DIP-14_W7.62mm
- U5: value 74HCT32 -> 74LS32; footprint Housings_DIP:DIP-14_W7.62mm -> Custom KiCad Library:DIP-14_W7.62mm
- U7: value 74HCT138 -> 74LS138; footprint Housings_DIP:DIP-16_W7.62mm -> Custom KiCad Library:DIP-16_W7.62mm
- U9: footprint Housings_DIP:DIP-28_W15.24mm_Socket -> Custom KiCad Library:DIP-28_W15.24mm_Socket
- moved C12 85.8 mm to (198.4, 118.4)
- moved C8 52.1 mm to (138.3, 81.7), turned to 0 degrees
- moved U10 50.3 mm to (144.5, 107.1), turned to 180 degrees
- moved C13 38.7 mm to (163.7, 135.4), turned to 0 degrees
- moved C3 38.2 mm to (125.5, 138.8), turned to 0 degrees
- moved U8 36.2 mm to (182.6, 107.1), turned to 180 degrees
- moved U1 36.0 mm to (144.5, 136.3), turned to 180 degrees
- moved C2 35.7 mm to (138.2, 138.8), turned to 0 degrees
- moved U7 35.3 mm to (182.6, 131.2), turned to 180 degrees
- moved C4 35.0 mm to (150.9, 138.8), turned to 0 degrees
- moved U11 31.4 mm to (157.2, 136.3), turned to 180 degrees
- moved U2 30.0 mm to (131.8, 136.3), turned to 180 degrees
- moved RP2 28.7 mm to (153.8, 78.6)
- moved SW2 27.4 mm to (150.0, 68.7)
- moved C10 26.7 mm to (176.3, 134.0), turned to 0 degrees
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Connections:
- U4 pad 13: Net-(U4-Pad13) -> Net-(U4-Pad10)
- U4 pad 4: Net-(U4-Pad11) -> Net-(U4-Pad4)
- U4 pad 5: Net-(U4-Pad10) -> Net-(U4-Pad4)
- U4 pad 6: IOR_DELAYED -> Net-(U4-Pad6)
- U4 pad 8: Net-(U4-Pad13) -> IOR_DELAYED
- U4 pad 9: Net-(U4-Pad9) -> Net-(U4-Pad6)
- U5 pad 11: Net-(U4-Pad9) -> Net-(U4-Pad11)
Routing:
- net VCC: track 443.8 -> 655.2 mm, vias 1 -> 0
- net GND: track 268.9 -> 83.3 mm, vias 0 -> 2
- net CS_ROM: track 33.7 -> 136.9 mm, vias 0 -> 1
- net A2: track 142.5 -> 190.7 mm, vias 1 -> 0
- net U1-Load: track 34.2 -> 82.4 mm, vias 2 -> 1
- net Net-(U3-Pad11): track 40.1 -> 85.9 mm
- net IOW: track 73.0 -> 113.7 mm
- net U2-OE: track 56.5 -> 97.1 mm
- net Net-(RP2-Pad7): track 53.8 -> 93.3 mm, vias 0 -> 2
- net A0: track 239.7 -> 200.5 mm
- net Net-(RP2-Pad8): track 55.4 -> 94.4 mm, vias 1 -> 0
- net Net-(R4-Pad2): track 74.9 -> 113.6 mm
- net D7: track 109.9 -> 71.7 mm, vias 0 -> 1
- net A16: track 98.2 -> 60.2 mm
- net Net-(U6-Pad9): track 46.9 -> 13.8 mm, vias 1 -> 0
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Other:
- net class 12V added: clearance 0.2, trace_width 1, via_dia 1, via_drill 0.6
- net class Default: clearance 0.2 -> 0.17
- net class Power removed
- rule pad_to_mask_clearance: 0.0508 -> 0
- rule trace_clearance: 0.2 -> 0.17
- board text added: "*Beware IC orientation*"
- board text added: "2 3 4 5 7"
- board text added: "Bootable 8-bit ISA IDE Interface"
- board text added: "IBM XT Slot-8 Mode (needs rear parts)"
- board text added: "IDE Address Switch"
- board text added: "IDE IRQ isn't supported in XT-IDE Universal BIOS as of R602. Leave unjumpered."
- board text added: "JLCJLCJLCJLC"
- board text added: "Monotech XT-IDE"
- board text added: "ROM Address Switch"
- board text added: "Rev 5.3"
- board text removed: "7 5 4 3 2"
- board text removed: "IBM XT Slot-8 Mode Needs rear SMD parts"
- board text removed: "IDE Address Switch Settings"
- board text removed: "IDE IRQ isn't supported in XT-IDE Universal BIOS as of R598. Leave unjumpered."
- board text removed: "Monotech XT-IDE Bootable 8-bit ISA IDE Interface"
- board text removed: "ROM Address Switch Settings"
- board text removed: "Rev 5.2"
