File: XT-IDE.sch (KiCad schematic (older format))
At the start: 49 parts, among them J1 Power output, J2 Conn_01x02, J3 External LED, J4 Conn_01x02, J5 Conn_02x05_Odd_Even, P6 CONN_1, P7 CONN_1, SW1 DIPS_06, SW2 DIPS_04, SW3 DPDT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

Commit message: Add files via upload
Update files to Rev5.1
Parts:
- BUS1: symbol BUSPC -> XT-IDE-rescue:BUSPC
- C1, C10, C11, C2, C3, C4, C5, C6, C7, C8, C9: footprint Capacitors_THT:C_Axial_L3.8mm_D2.6mm_P7.50mm_Horizontal -> Capacitors_THT:C_Rect_L7.0mm_W2.0mm_P5.00mm; symbol C -> Device:C
- C12: symbol CP -> Device:CP
- C13: symbol C -> Device:C
- D1: symbol LED-RESCUE-XT-IDE -> XT-IDE-rescue:LED-RESCUE-XT-IDE
- IDE1: symbol Conn_02x20_Odd_Even -> XT-IDE-rescue:Conn_02x20_Odd_Even
- J1: symbol Conn_01x04_Female -> XT-IDE-rescue:Conn_01x04_Female
- J2, J4: symbol Conn_01x02 -> XT-IDE-rescue:Conn_01x02
- J3: symbol CONN_2 -> XT-IDE-rescue:CONN_2
- J5: symbol Conn_02x05_Odd_Even -> XT-IDE-rescue:Conn_02x05_Odd_Even
- P6, P7: symbol CONN_1 -> XT-IDE-rescue:CONN_1
- R1, R2, R3, R4, R5, R6: symbol R -> Device:R
- RP1, RP2: symbol R_Network07 -> Device:R_Network07
- SW1: symbol SW_DIP_x06 -> XT-IDE-rescue:SW_DIP_x06
- SW2: symbol SW_DIP_x04 -> XT-IDE-rescue:SW_DIP_x04
- SW3: footprint Custom:CKCOMP-OS203011MS1QP1 -> Custom:CKCOMP-OS202011MA0QS1; symbol SW_DPDT_x2 -> XT-IDE-rescue:SW_DPDT_x2
- SW4: symbol SW_DPDT_x2 -> XT-IDE-rescue:SW_DPDT_x2
- SW5, SW6: symbol SW_SPDT -> XT-IDE-rescue:SW_SPDT
- U1, U2: symbol 74LS573 -> XT-IDE-rescue:74LS573
- U10, U8: symbol 74LS688 -> XT-IDE-rescue:74LS688
- U11, U3: symbol 74LS245 -> XT-IDE-rescue:74LS245
- U12: symbol 74LS33 -> XT-IDE-rescue:74LS33
- U4, U6: symbol 74LS04 -> XT-IDE-rescue:74LS04
- U5: symbol 74LS32 -> XT-IDE-rescue:74LS32
- U7: symbol 74LS138 -> XT-IDE-rescue:74LS138
- U9: symbol 28C256-RESCUE-XT-IDE -> XT-IDE-rescue:28C256-RESCUE-XT-IDE
Connections:
- wire segments 182 -> 243

Commit message: Add files via upload
Parts:
- C1, C10, C11, C13, C2, C3, C4, C5, C6, C7, C8, C9: value C -> 0.1uF
- IDE1: footprint Custom:Pin_Header_Angled_2x20_ShortSilkS -> Custom:Pin_Header_Angled_2x20_Pitch2.54mm_Shrouded
- RP1, RP2: value 10k -> 10K
- SW1: value DIPS_06 -> IDE Address; footprint Buttons_Switches_THT:SW_DIP_x6_W7.62mm_Slide -> Buttons_Switches_THT:SW_DIP_x6_W7.62mm_Slide_LowProfile
- SW2: value DIPS_04 -> ROM Address; footprint Buttons_Switches_THT:SW_DIP_x4_W7.62mm_Slide -> Buttons_Switches_THT:SW_DIP_x4_W7.62mm_Slide_LowProfile
- U9: value 28C256 -> 28C64B/28C256
Connections:
- net ROM_WE: now also SW6.3 (C); no longer SW6.1 (A)
- net at SW1.7, U8.14 (R5): now also RP1.7 (R6); no longer RP1.8 (R7)
- net at SW1.8, U8.16 (R6): now also RP1.6 (R5); no longer RP1.7 (R6)
- net at SW1.9, U8.18 (R7): now also RP1.5 (R4); no longer RP1.6 (R5)
- net at SW1.12, U8.3 (R0): now also RP1.2 (R1); no longer RP1.3 (R2)
- net at SW1.11, U8.5 (R1): now also RP1.3 (R2); no longer RP1.4 (R3)
- net at SW1.10, U8.7 (R2): now also RP1.4 (R3); no longer RP1.5 (R4)
Other:
- note added: "IDE ACTIVITY LEDS"
- note added: "ROM Address Notes:\nFor full 32K device (28C256) set SW4 to ON, and SW2 (3 and 4) to OFF\nFor 8K device (28C64B) set SW4 to OFF"
- note added: "Switch Settings\nSW2 1-4: ROM Address (ON == 1)\nSW4: 8K Mode (ON == enabled)\nSW5: ROM Enable (ON == enabled)\nSW6: ROM Write-Protect (ON == enabled)"
- note removed: "ALL CAPS MARKED C ARE 0.01 - 0.1 uF BYPASS"
- note removed: "IDE ACTIVITY LEDS\nOBSERVE POLARITY -- PIN 1 CATHODE"
- note removed: "ROM Address Notes:\nFor full 32K device (28C256) set SW4, and SW2 (3 and 4) to OFF\nFor 8K device (28C64B) set SW4 ON\nSW2 (3 and 4) become address switches"
- note removed: "Switch Settings\nSW2 1-4: ROM Address (ON == 1)\nSW4: 8K Mode (ON == enabled)\nSW5: ROM Enable (ON == enabled)\nSW6: Write Enable (ON == enabled)"
- moved on the sheet: C1, C10, C11, C12, C13, C2, C3, C4, C5, C6, C7, C8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

Commit message: Add files via upload
Parts:
- SW1: footprint Buttons_Switches_THT:SW_DIP_x6_W7.62mm_Slide_LowProfile -> Buttons_Switches_THT:SW_DIP_x6_W7.62mm_Slide
- SW2: footprint Buttons_Switches_THT:SW_DIP_x4_W7.62mm_Slide_LowProfile -> Buttons_Switches_THT:SW_DIP_x4_W7.62mm_Slide
Changed lines of the file:
@@
 F 0 "SW2" H 1500 9400 60  0000 C CNN
 F 1 "ROM Address" V 1500 9150 60  0001 C CNN
-F 2 "Buttons_Switches_THT:SW_DIP_x4_W7.62mm_Slide_LowProfile" H 1250 9150 60  0001 C CNN
+F 2 "Buttons_Switches_THT:SW_DIP_x4_W7.62mm_Slide" H 1250 9150 60  0001 C CNN
 F 3 "" H 1250 9150 60  0001 C CNN
 	1    1250 9150
@@
 F 0 "SW1" H 1500 5650 60  0000 C CNN
 F 1 "IDE Address" V 1600 5300 60  0001 C CNN
-F 2 "Buttons_Switches_THT:SW_DIP_x6_W7.62mm_Slide_LowProfile" H 1250 5300 60  0001 C CNN
+F 2 "Buttons_Switches_THT:SW_DIP_x6_W7.62mm_Slide" H 1250 5300 60  0001 C CNN
 F 3 "" H 1250 5300 60  0001 C CNN
 	1    1250 5300

Commit message: Updated to Rev5.3
Parts:
- added C13: 10uF, Capacitor_THT:CP_Radial_Tantal_D4.5mm_P5.00mm, symbol Device:CP
- C1, C10, C11, C2, C3, C4, C5, C6, C7, C8, C9: value 0.1uF -> 100nF; footprint Capacitors_THT:C_Rect_L7.0mm_W2.0mm_P5.00mm -> Capacitor_THT:C_Disc_D4.3mm_W1.9mm_P5.00mm
- C12: renamed from C13; value 0.1uF -> 100nF; footprint Resistors_SMD:R_0805_HandSoldering -> Capacitor_SMD:C_0805_2012Metric_Pad1.15x1.40mm_HandSolder
- C14: renamed from C12; value 47uF -> 10uF; footprint Capacitors_THT:CP_Radial_D6.3mm_P2.50mm -> Capacitor_THT:CP_Radial_Tantal_D4.5mm_P5.00mm
- D1: footprint LEDs:LED_D5.0mm -> LED_THT:LED_D5.0mm
- J1: footprint Pin_Headers:Pin_Header_Angled_1x04_Pitch2.54mm -> Connector_PinHeader_2.54mm:PinHeader_1x04_P2.54mm_Horizontal
- J2, J4: footprint Pin_Headers:Pin_Header_Straight_1x02_Pitch2.54mm -> Connector_PinHeader_2.54mm:PinHeader_1x02_P2.54mm_Vertical
- J3: footprint Pin_Headers:Pin_Header_Angled_1x02_Pitch2.54mm -> Connector_PinHeader_2.54mm:PinHeader_1x02_P2.54mm_Horizontal
- J5: footprint Pin_Headers:Pin_Header_Straight_2x05_Pitch2.54mm -> Connector_PinHeader_2.54mm:PinHeader_2x05_P2.54mm_Vertical
- P6, P7: footprint Mounting_Holes:MountingHole_3mm -> MountingHole:MountingHole_3.2mm_M3
- R1, R2, R3, R4: footprint Resistors_THT:R_Axial_DIN0207_L6.3mm_D2.5mm_P7.62mm_Horizontal -> Resistor_THT:R_Axial_DIN0207_L6.3mm_D2.5mm_P7.62mm_Horizontal
- R5, R6: footprint Resistors_SMD:R_0805_HandSoldering -> Resistor_SMD:R_0805_2012Metric_Pad1.15x1.40mm_HandSolder
- RP1, RP2: footprint Resistors_THT:R_Array_SIP8 -> Resistor_THT:R_Array_SIP9
- SW1: footprint Buttons_Switches_THT:SW_DIP_x6_W7.62mm_Slide -> Button_Switch_THT:SW_DIP_SPSTx06_Slide_9.78x17.42mm_W7.62mm_P2.54mm
- SW2: footprint Buttons_Switches_THT:SW_DIP_x4_W7.62mm_Slide -> Button_Switch_THT:SW_DIP_SPSTx04_Slide_9.78x12.34mm_W7.62mm_P2.54mm
- SW5, SW6: footprint Custom:CKCOMP-OS102011MA1QN1 -> Button_Switch_THT:SW_CuK_OS102011MA1QN1_SPDT_Angled
- U1, U2: value 74HCT573 -> 74LS573; footprint Housings_DIP:DIP-20_W7.62mm -> Custom KiCad Library:DIP-20_W7.62mm
- U10, U8: value 74HCT688 -> 74LS688; footprint Housings_DIP:DIP-20_W7.62mm -> Custom KiCad Library:DIP-20_W7.62mm
- U11, U3: value 74HCT245 -> 74LS245; footprint Housings_DIP:DIP-20_W7.62mm -> Custom KiCad Library:DIP-20_W7.62mm
- U12: footprint Housings_SOIC:SOIC-14_3.9x8.7mm_Pitch1.27mm -> Custom KiCad Library:SOIC-14_3.9x8.7mm_P1.27mm
- U4, U6: value 74HCT04 -> 74LS04; footprint Housings_DIP:DIP-14_W7.62mm -> Custom KiCad Library:DIP-14_W7.62mm
- U5: value 74HCT32 -> 74LS32; footprint Housings_DIP:DIP-14_W7.62mm -> Custom KiCad Library:DIP-14_W7.62mm
- U7: value 74HCT138 -> 74LS138; footprint Housings_DIP:DIP-16_W7.62mm -> Custom KiCad Library:DIP-16_W7.62mm
- U9: footprint Housings_DIP:DIP-28_W15.24mm_Socket -> Custom KiCad Library:DIP-28_W15.24mm_Socket
Connections:
- net GND: now also C13.2
- net IOR_DELAYED: now also U4.8; no longer U4.6
- net VCC: now also C13.1
- net at U5.11: now also U4.11; no longer U4.9
- net at U4.4: now also U4.5; no longer U4.11
- net at U4.10: now also U4.13; no longer U4.5
- new net: U4.6, U4.9
Other:
- moved on the sheet: U4C, U4D, U4E
