File: XT-IDE Deluxe.kicad_sch (KiCad schematic)
At the start: 58 parts, among them J1 IDE, J10 IRQ5, J11 IRQ7, J2 CF_Adapter, J3 IDE IRQ, J4 VCC, J5 Power Output, J6 MemExp, J7 IRQ2, J8 IRQ3, J9 IRQ4, SW1 HiSpeed, SW2 Config, U1 HCT245, U10 F138, U12 HCT02, U13 AHC1G09, U14 F138, U15 HCT86, U16 F138, U2 HCT573, U3 HCT573, U4 HCT245, U5 HCT04, U6 HCT32, U7 HCT04, U8 28C256, U9 HCT86

Commit message: Update to v1.2.
Parts:
- removed F1, F2: 1.5A, Fuse:Fuse_1206_3216Metric, symbol Device:Fuse
- removed H1, H2, H3, H4: M3, MountingHole:MountingHole_3.2mm_M3_Pad, symbol Mechanical:MountingHole_Pad
- removed H5: MountingHole, MountingHole:MountingHole_3.2mm_M3, symbol Mechanical:MountingHole
- removed J2: CF_Adapter, Connector_PinSocket_2.54mm:PinSocket_2x20_P2.54mm_Vertical, symbol Connector_Generic:Conn_02x20_Odd_Even
- removed J4: VCC, Connector_PinHeader_2.54mm:PinHeader_1x01_P2.54mm_Vertical, symbol Connector:Conn_01x01_Male
- removed JP1: 5V on IDE Pin20, Connector_PinHeader_2.54mm:PinHeader_1x02_P2.54mm_Vertical, symbol Device:Jumper
- removed SW2: Config, Button_Switch_THT:SW_DIP_SPSTx12_Slide_9.78x32.66mm_W7.62mm_P2.54mm, symbol Switch:SW_DIP_x12
- removed U13: AHC1G09, Package_TO_SOT_SMD:SOT-353_SC-70-5, symbol 74xGxx:74AHC1G08
- removed U8: 28C256, Package_DIP:DIP-28_W15.24mm_Socket, symbol Memory_EEPROM:28C256
- added C13: 100nF, Capacitor_SMD:C_0603_1608Metric, symbol Device:C_Small
- added D3: BAT54A, Package_TO_SOT_SMD:SOT-23, symbol Diode:BAT54A
- added F1, F2: 1.5A, Fuse:Fuse_1812_4532Metric, symbol Device:Polyfuse
- added H1, H2: MountingHole, MountingHole:MountingHole_3.2mm_M3, symbol Mechanical:MountingHole
- added J2: CF Slot, Custom:CF_Slot_UMax_CFH-R3C1LBMXXMN2, symbol compactflash_connector:CF Slot
- added JP1: ROM Type, Custom:PinHeader_2x04_P2.54mm_Vertical_SMD, symbol Connector_Generic:Conn_02x04_Odd_Even
- added R3: 220, Resistor_SMD:R_0805_2012Metric, symbol Device:R
- added SW1: Config, Button_Switch_SMD:SW_DIP_SPSTx12_Slide_6.7x32.04mm_W8.61mm_P2.54mm_LowProfile, symbol Switch:SW_DIP_x12
- added SW3: 5V on IDE Pin20, Custom:SW_DPDT_MS-22D28-G020, symbol Switch:SW_SPST
- added U8: ROM, Custom:DIP-32_W16.51mm_SMDSocket_LongPads, symbol Memory_Flash:SST39SF040
- BUS1: value Bus_ISA_8bit -> 8-bit ISA
- C1, C2: value 106 -> 10uF; footprint Capacitor_SMD:C_0805_2012Metric -> Capacitor_SMD:C_0603_1608Metric
- C10, C11, C12, C3, C4, C5, C6, C7, C8, C9: value 104 -> 100nF; footprint Capacitor_SMD:C_0805_2012Metric -> Capacitor_SMD:C_0603_1608Metric
- D1: value LED -> Rear LED; footprint LED_SMD:LED_0805_2012Metric -> Custom:3mm_LED_RightAngle
- D2: value LED -> LED Header
- J1: footprint Connector_IDC:IDC-Header_2x20_P2.54mm_Horizontal -> Custom:IDC-20_P2.54mm_Vertical_SMD
- J6: footprint Connector_PinHeader_2.54mm:PinHeader_2x17_P2.54mm_Vertical -> Custom:MicroRAM_Expansion; symbol Connector_Generic:Conn_02x17_Odd_Even -> Connector_Generic:Conn_02x20_Odd_Even
- LOGO1: footprint (none) -> Custom KiCad Library:Monotech Logo 12mm
- R1, R2: value 1k -> 220
- SW2: renamed from SW1; value HiSpeed -> Rev2; footprint Button_Switch_THT:SW_CuK_JS202011CQN_DPDT_Straight -> Custom:SW_DPDT_MS-22D28-G020
- U1, U4: footprint Package_SO:TSSOP-20_4.4x6.5mm_P0.65mm -> Custom KiCad Library:TSSOP-20_4.4x6.5mm_P0.65mm
- U10, U14, U16: value F138 -> AHCT138; footprint Package_SO:SOIC-16_3.9x9.9mm_P1.27mm -> Custom KiCad Library:SOIC-16_3.9x9.9mm_P1.27mm
- U12, U15, U5, U6, U7, U9: footprint Package_SO:SOIC-14_3.9x8.7mm_P1.27mm -> Custom KiCad Library:SOIC-14_3.9x8.7mm_P1.27mm
- U2, U3: footprint Package_SO:SOIC-20W_7.5x12.8mm_P1.27mm -> Custom KiCad Library:TSSOP-20_4.4x6.5mm_P0.65mm
Connections:
- net +12V: now also F2.2
- net 5V_Fused: now also C3.1, J1.29 (Pin_29), F1.1, J2.13 (VCC), J2.36 (~{WE}), J2.38 (VCC), J2.44 (~{REG}), SW3.1 (A)
- net A0: now also U8.12 (A0)
- net A1: now also U8.11 (A1)
- net A10: now also U8.23 (A10)
- net A11: now also U8.25 (A11)
- net A12: now also U8.4 (A12)
- net A13: now also JP1.7 (Pin_7), U8.28 (A13)
- net A14: now also JP1.4 (Pin_4)
- net A2: now also U8.10 (A2)
- net A3: now also U8.9 (A3)
- net A4: now also U8.8 (A4)
- net A5: now also U8.7 (A5)
- net A6: now also U8.6 (A6)
- net A7: now also U8.5 (A7)
- net A8: now also U8.27 (A8)
- net A9: now also U8.26 (A9)
- net AEN: now also SW1.9
- net BA1: now also J2.19 (A1)
- net BA2: now also J2.18 (A2)
- net D0: now also U1.2 (A0), U8.13 (D0); no longer U1.9 (A7)
- net D1: now also U1.3 (A1), U8.14 (D1); no longer U1.8 (A6)
- net D2: now also U1.4 (A2), U8.15 (D2); no longer U1.7 (A5)
- net D3: now also U1.5 (A3), U8.17 (D3); no longer U1.6 (A4)
- net D4: now also U1.6 (A4), U8.18 (D4); no longer U1.5 (A3)
- net D5: now also U1.7 (A5), U8.19 (D5); no longer U1.4 (A2)
- net D6: now also U1.8 (A6), U8.20 (D6); no longer U1.3 (A1)
- net D7: now also U1.9 (A7), U8.21 (D7); no longer U1.2 (A0)
- net DB0: now also U1.18 (B0), U2.2 (D0), J2.21 (D0); no longer U1.11 (B7), U2.9 (D7)
- net DB1: now also U1.17 (B1), U2.3 (D1), J2.22 (D1); no longer U1.12 (B6), U2.8 (D6)
- net DB10: now also U2.17 (Q2), J2.49 (D10); no longer U2.14 (Q5)
- net DB11: now also U2.16 (Q3), J2.27 (D11); no longer U2.15 (Q4)
- net DB12: now also U2.15 (Q4), J2.28 (D12); no longer U2.16 (Q3)
- net DB13: now also U2.14 (Q5), J2.29 (D13); no longer U2.17 (Q2)
- net DB14: now also U2.13 (Q6), J2.30 (D14); no longer U2.18 (Q1)
- net DB15: now also U2.12 (Q7), J2.31 (D15); no longer U2.19 (Q0)
- net DB2: now also U1.16 (B2), U2.4 (D2), J2.23 (D2); no longer U1.13 (B5), U2.7 (D5)
- net DB3: now also U1.15 (B3), U2.5 (D3), J2.2 (D3); no longer U1.14 (B4), U2.6 (D4)
- net DB4: now also U1.14 (B4), U2.6 (D4), J2.3 (D4); no longer U1.15 (B3), U2.5 (D3)
- net DB5: now also U1.13 (B5), U2.7 (D5), J2.4 (D5); no longer U1.16 (B2), U2.4 (D2)
- net DB6: now also U1.12 (B6), U2.8 (D6), J2.5 (D6); no longer U1.17 (B1), U2.3 (D1)
- net DB7: now also U1.11 (B7), U2.9 (D7), J2.6 (D7); no longer U1.18 (B0), U2.2 (D0)
- net DB8: now also U2.19 (Q0), J2.47 (D8); no longer U2.12 (Q7)
- net DB9: now also U2.18 (Q1), J2.48 (D9); no longer U2.13 (Q6)
- net GND: now also C13.2, J2.0 (Shield), J2.1 (GND), J2.10 (A9), J2.11 (A8), J2.12 (A7), J2.14 (A6), J2.15 (A5), J2.16 (A4), J2.17 (A3), J2.25 (~{CD2}), J2.26 (~{CD1}), J2.50 (GND), J2.8 (A10), J2.9 (~{ATASEL}), R3.1, SW1.1, SW1.12, U8.16 (GND); no longer R1.1, R2.1, RN1.7 (R2.2)
- net IDE_A5: now also RN3.3 (R3.1), SW1.21; no longer RN3.4 (R4.1)
- net IDE_A6: now also RN3.2 (R2.1), SW1.22; no longer RN3.3 (R3.1)
- net IDE_A7: now also SW1.23
- net IDE_IRQ: now also J2.37 (INTRQ)
- net IRQ2: now also J6.37 (Pin_37)
- net IRQ3: now also J6.40 (Pin_40)
- net IRQ5: now also J6.39 (Pin_39)
- net ROM_A13: now also RN2.3 (R3.1), SW1.17; no longer RN2.4 (R4.1)
- net ROM_A14: now also RN2.2 (R2.1), SW1.18; no longer RN2.3 (R3.1)
- net ROM_A15: now also RN2.1 (R1.1), SW1.19; no longer RN2.2 (R2.1)
- net ROM_A16: now also RN3.4 (R4.1), SW1.20; no longer RN2.1 (R1.1)
- net RST: now also J6.38 (Pin_38)
- net VCC: now also RN1.7 (R2.2), C13.1, F1.2, JP1.1 (Pin_1), SW1.2, SW1.3, SW1.4, SW1.5, SW1.6, SW1.7, SW1.8, U8.1 (A18), U8.2 (A16), U8.30 (A17), U8.32 (VCC); no longer C3.1, J1.29 (Pin_29)
- net ~{BIOR}: now also J2.34 (~{IORD})
- net ~{BIOW}: now also J2.35 (~{IOWR})
- net ~{BRST}: now also J2.41 (~{RESET})
- net ~{CS1}: now also J2.7 (~{CS0})
- net ~{CS3}: now also J2.32 (~{CS1})
- net ~{DASP}: now also RN1.4 (R4.1), J2.45 (~{DASP})
- net ~{IOR_DELAY}: now also U5.6; no longer U5.12
- net ~{IOR}: now also J6.35 (Pin_35), U5.1; no longer U5.5
- net ~{IOW}: now also J6.36 (Pin_36)
- net ~{MEMR}: now also U8.24 (OE)
- net ~{MEMW}: now also SW1.10
- net ~{PDIAG}: now also J2.46 (~{PDIAG})
- net ~{ROM_CS}: now also U8.22 (CE)
- net ~{ROM_EN}: now also RN1.2 (R2.1), SW1.16; no longer RN1.3 (R3.1)
- net ~{ROM_WR}: now also RN1.3 (R3.1), JP1.5 (Pin_5), SW1.15, U8.31 (PGM); no longer RN1.4 (R4.1)
- net ~{Slot8}: now also SW1.11
- net ~{xSlot8}: now also D3.3, SW1.14
- net at U6.2: now also U5.8; no longer U5.2
- net at U6.8: now also D3.2
- net at U6.11: now also D3.1
- net A3Compat_A0Speed: now reaches U5.9
- net A3Compat_A0Speed: now also SW2.2 (B), U10.3 (A2), U6.4; no longer U5.6
- net at U5.11: now also U5.12; no longer U5.8
- net at U5.13: now also U5.2; no longer U5.10
- net at D1.1 (K): now also R2.2; no longer R1.2
- net at D2.1 (K): now also R3.2; no longer R2.2
- net 12V_Fused: now reaches J5.4 (Pin_4)
- net 12V_Fused: now also F2.1
- net A0-OR-3 renamed A0Compat_A3Speed
- removed net A3-OR-0: SW2.2 (B), U10.3 (A2), U5.1, U6.4
- net BA0-OR-BA3 renamed B_A0_A3
- net B_A0_A3: now also J2.20 (A0)
- net IDE_5V renamed IDE_pin20
- net IDE_pin20: now also SW3.2 (B)
- net ROM_8K_1 renamed Dec_A13
- net Dec_A13: now also U15.13, JP1.8 (Pin_8); no longer U15.10
- removed net ROM_8K_2: RN1.2 (R2.1), U15.13
- net ~{LA1-OE} renamed ~{LA1_OE}
- net ~{LA2-OE} renamed ~{LA2_OE}
- net ~{xLA2-OE} renamed ~{xLA2_OE}
- new net: U5.10, U5.5
- new net: R1.1, U8.3 (A15)
- new net: JP1.2 (Pin_2), R1.2
- new net: JP1.3 (Pin_3), U8.29 (A14)
- new net Dec_A14: JP1.6 (Pin_6), RN2.4 (R4.1), U15.10
- new net ~{Master}: J2.39 (~{CSEL}), SW1.24
- new net ~{RearLED_En}: R2.1, SW1.13
Other:
- note added: "! = Default * = All ROM support ^ = 16K/8K ROM support = 8K ROM support JP1: ROM Type: 27/28(C)64 : 1-2, 3-5, 4-6, 7-8 27(C)128 : 1-2, 3-5, 4-6 27(C)256/512: 1-2, 3-4 (and 32-pin ROMs) 28C256 : 2-4, 3-5 With chips >32K, only the topmost 32K segment is used."
- note added: "2764/27128/27256/27512/27010/27020/27040 Writeable: 28C64/28C256/SST39SF0*0"
- note added: "For machines such as PS/2 Model 30(-286)."
- note added: "Littelfuse 1812L150/16"
- note added: "Pads for jumper wire if IRQ support is needed in future"
- note added: "ROM, LEDs, Slot8"
- note added: "SW1: Config: ============ Switch 1: CF Slot: ON = Master, OFF = Slave (only relevant if a CF card is inserted) Switches 2-4: IDE I/O Address 234 IDE 000 300 ! 001 320 010 340 011 360 100 380 101 3A0 110 3C0 111 3E0 Switches 5-8: ROM Memory Address 5678 ROM 0000 C0000* 0001 C2000 0010 C4000 ^ 0011 C6000 0100 C8000* 0101 CA000 0110 CC000 ^ 0111 CE000 1000 D0000* ! 1001 D2000 1010 D4000 ^ 1011 D6000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"
- note added: "SW2: XT-IDE Rev1/Rev2 Mode ("Rev2" is also known as HiSpeed mode or Chuck(G) mod) SW3: Put 5V on IDE pin 20, intended for CF adapters and DoMs."
- note added: "Schematic default state shows Rev1 mode"
- note added: "UMax CFH-R3C1LBMXXMN2"
- note removed: "IDE Address: 123 IDE 000 300 ! 001 320 010 340 011 360 100 380 101 3A0 110 3C0 111 3E0 ! = Default * = All ROM support ^ = 16K/8K ROM support = 8K ROM support ROM Size: 89 11 = 8K: 27(C)64, 28C64 10 = 16K: 27C128 00 = 32K: 28C256 (not 27C256) 10: ROM Enable 11: ROM Write Enable 12: IBM XT Slot-8 Mode"
- note removed: "ROM Address: 4567 ROM 0000 C0000* 0001 C2000 0010 C4000 ^ 0011 C6000 0100 C8000* 0101 CA000 0110 CC000 ^ 0111 CE000 1000 D0000* ! 1001 D2000 1010 D4000 ^ 1011 D6000 1100 D8000* 1101 DA000 1110 DC000 ^ 1111 DE000"
- note removed: "ROM, LED, Slot8"
- title: XT-IDE Deluxe -> XT-IDE Deluxe (8-bit ISA Bootable IDE+CF Interface)
- moved on the sheet: C1, C10, C11, C12, C2, C3, C4, C5, C6, C7, C8, C9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
